File: hardware/prototype6/edrumulus.kicad_sch (KiCad schematic)
At the start: 106 parts, among them J1 Hi-Hat, J10 MIDI-IN, J11 MIDI-OUT, J2 Snare, J3 Crash, J4 Ride, J5 Tom1, J6 Tom2, J7 Tom3, J8 Kick, J9 Hi-Hat-Ctrl, U1 ESP32-DEVKIT-V1, U2 6N138, U3 L78L33_TO92

Commit message: more routing for prototype 6
Connections:
- net 3V3: no longer R41.1, R42.2, U2.8 (VCC)
- net ESP-3V3: now reaches U1.16 (3V3)
- net ESP-3V3: now also R41.1, R42.2, U2.8 (VCC)
- no-connect marks 21 -> 20
Changed lines of the file:
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@@
   (no_connect (at 160.528 52.07))
   (no_connect (at 191.77 97.79))
-  (no_connect (at 191.77 107.95))
   (no_connect (at 137.668 25.4))
   (no_connect (at 191.77 90.17))
@@
     )
   )
+  (global_label "ESP-3V3" (shape input) (at 191.77 107.95 0) (fields_autoplaced)
+    (effects (font (size 1.27 1.27)) (justify left))
+    (property "Referenzen zwischen Schaltplänen" "${INTERSHEET_REFS}" (id 0) (at 202.8028 107.8706 0)
+      (effects (font (size 1.27 1.27)) (justify left) hide)
+    )
+  )
   (global_label "3V3" (shape input) (at 76.708 107.696 0) (fields_autoplaced)
     (effects (font (size 1.27 1.27)) (justify left))
@@
     )
   )
-  (global_label "3V3" (shape input) (at 188.468 54.61 0) (fields_autoplaced)
-    (effects (font (size 1.27 1.27)) (justify left))
-    (property "Referenzen zwischen Schaltplänen" "${INTERSHEET_REFS}" (id 0) (at -28.702 -44.45 0)
-      (effects (font (size 1.27 1.27)) hide)
+  (global_label "ESP-3V3" (shape input) (at 188.468 54.61 0) (fields_autoplaced)
+    (effects (font (size 1.27 1.27)) (justify left))
+    (property "Referenzen zwischen Schaltplänen" "${INTERSHEET_REFS}" (id 0) (at 199.5008 54.5306 0)
+      (effects (font (size 1.27 1.27)) (justify left) hide)
     )
   )
@@
     )
   )
-  (global_label "3V3" (shape input) (at 178.308 24.13 180) (fields_autoplaced)
-    (effects (font (size 1.27 1.27)) (justify right))
-    (property "Referenzen zwischen Schaltplänen" "${INTERSHEET_REFS}" (id 0) (at -28.702 -44.45 0)
-      (effects (font (size 1.27 1.27)) hide)
-    )
-  )
   (global_label "UART_RX" (shape input) (at 197.358 39.37 180) (fields_autoplaced)
     (effects (font (size 1.27 1.27)) (justify right))
@@
     (property "Referenzen zwischen Schaltplänen" "${INTERSHEET_REFS}" (id 0) (at 5.842 -49.149 0)
       (effects (font (size 1.27 1.27)) hide)
+    )
+  )
+  (global_label "ESP-3V3" (shape input) (at 178.308 24.13 180) (fields_autoplaced)
+    (effects (font (size 1.27 1.27)) (justify right))
+    (property "Referenzen zwischen Schaltplänen" "${INTERSHEET_REFS}" (id 0) (at 167.2752 24.2094 0)
+      (effects (font (size 1.27 1.27)) (justify right) hide)
     )
   )
@@
   (symbol (lib_id "Isolator:6N138") (at 173.228 34.29 0) (unit 1)
     (in_bom yes) (on_board yes)
-    (property "Reference" "U2" (id 0) (at 168.402 22.098 0))
-    (property "Value" "6N138" (id 1) (at 168.402 24.638 0))
+    (property "Reference" "U2" (id 0) (at 179.832 42.672 0))
+    (property "Value" "6N138" (id 1) (at 164.592 42.418 0))
     (property "Footprint" "Package_DIP:DIP-8_W7.62mm_Socket" (id 2) (at 180.594 41.91 0)
       (effects (font (size 1.27 1.27)) hide)
