File: hardware/prototype6/edrumulus.kicad_pcb (KiCad board)
At the start: 2 copper layers, 196.7 x 84.6 mm, 106 parts, among them J1 Hi-Hat, J10 MIDI-IN, J11 MIDI-OUT, J2 Snare, J3 Crash, J4 Ride, J5 Tom1, J6 Tom2, J7 Tom3, J8 Kick, J9 Hi-Hat-Ctrl, U1 ESP32-DEVKIT-V1, U2 6N138, U3 L78L33_TO92

Commit message: more routing for prototype 6
Connections:
- R41 pad 1: 3V3 -> ESP-3V3
- R42 pad 2: 3V3 -> ESP-3V3
- U1 pad 16: unconnected-(U1-Pad16) -> ESP-3V3
- U2 pad 8: 3V3 -> ESP-3V3
Routing:
- net GND: track 41.7 -> 793.5 mm
- net 3V3: track 0.00 -> 299.7 mm
- net GPIO27: track 3.33 -> 175.8 mm
- net GPIO13: track 4.16 -> 157.7 mm
- net GPIO14: track 3.61 -> 145.3 mm
- net GPIO34: track 3.19 -> 117.3 mm
- net UART_TX: track 0.00 -> 95.0 mm, vias 0 -> 1
- net GPIO15: track 0.00 -> 83.0 mm
- net GPIO33: track 3.83 -> 80.1 mm
- net GPIO26: track 3.13 -> 79.2 mm
- net UART_RX: track 0.00 -> 74.6 mm, vias 0 -> 1
- net GPIO32: track 3.55 -> 75.1 mm
- net ESP-3V3: track 0.00 -> 65.9 mm
- net GPIO25: track 0.00 -> 65.0 mm
- net 5V: track 0.00 -> 64.1 mm
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
Commit message: prototype 6 fine tuning
Routing:
- net 3V3: track 299.7 -> 322.0 mm
- net GND: track 793.5 -> 798.8 mm
- net GPIO32: track 75.1 -> 79.1 mm
- net GPIO34: track 117.3 -> 119.5 mm

Commit message: more fine tuning and fixing for prototype 6
Routing:
- net GND: track 798.8 -> 806.3 mm
- net GPIO15: track 83.0 -> 87.5 mm
- net RIDE-RING: track 31.0 -> 35.4 mm
- net GPIO32: track 79.1 -> 77.0 mm
- net GPIO35: track 54.7 -> 56.4 mm
- net GPIO39: track 45.1 -> 43.8 mm
- net CRASH1-RING: track 25.8 -> 26.7 mm
- net GPIO27: track 175.8 -> 176.6 mm

Commit message: finished prototype 6
Routing:
- net GPIO27: track 176.6 -> 153.8 mm
- net GPIO13: track 157.7 -> 153.8 mm
- net GPIO14: track 145.1 -> 141.3 mm
- net GPIO25: track 65.4 -> 68.6 mm
- net GPIO26: track 79.6 -> 81.2 mm
- net 3V3: track 321.6 -> 322.2 mm
- added copper zone on B.Cu, net GND
- added copper zone on F.Cu, net GND
Other:
- board text added: "Edrumulus Prototype 6"

Commit message: use lower resistors for MIDI out because we have 3.3V
Parts:
- R39: value 220 -> 10
- R41: value 220 -> 33
Changed lines of the file:
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@@
       (effects (font (size 1 1) (thickness 0.15)))
     )
-    (fp_text value "220" (at 0.508 -2.54) (layer "F.SilkS")
+    (fp_text value "10" (at 0.508 -2.54) (layer "F.SilkS")
       (effects (font (size 1 1) (thickness 0.15)))
     )
@@
       (effects (font (size 1 1) (thickness 0.15)))
     )
-    (fp_text value "220" (at 10.498668 -2.483497) (layer "F.SilkS")
-      (effects (font (size 1 1) (thickness 0.15)))
-    )
+    (fp_text value "33" (at 10.498668 -2.483497) (layer "F.SilkS")
+      (effects (font (size 1 1) (thickness 0.15)))
+    )
